Commit message: my xacro

File: neuronbot2_description/urdf/accessories/sensor_arch.urdf.xacro (robot description, xacro)
@@ -7,5 +7,5 @@
              <visual>
                  <geometry>
-                     <mesh filename="package://husky_description/meshes/accessories/${size}_mm_sensor_arch.dae" />
+                     <mesh filename="package://neuronbot2_description/meshes/neuronbot2/accessories/${size}_mm_sensor_arch.dae" />
                  </geometry>
              </visual>
@@ -13,5 +13,5 @@
                  <origin xyz="0 0 0" rpy="0 0 0"/>
                  <geometry>
-                     <mesh filename="package://husky_description/meshes/accessories/${size}_mm_sensor_arch.dae" />
+                     <mesh filename="package://neuronbot2_description/meshes/neuronbot2/accessories/${size}_mm_sensor_arch.dae" />
                  </geometry>
              </collision>

File: neuronbot2_description/urdf/accessories/sick_lms1xx_mount.urdf.xacro (robot description, xacro)
@@ -33,5 +33,5 @@
         <geometry>
           <!-- Origin of this mesh is the base of the bracket. -->
-          <mesh filename="package://husky_description/meshes/accessories/lms1xx_mount.dae" />
+          <mesh filename="package://neuronbot2_description/meshes/neuronbot2/accessories/lms1xx_mount.dae"/>
         </geometry>
       </visual>

File: neuronbot2_description/urdf/decorations.urdf.xacro (robot description, xacro)
@@ -16,5 +16,5 @@
         <origin xyz="0 0 0" rpy="0 0 0" />
         <geometry>
-          <mesh filename="package://husky_description/meshes/top_chassis.dae" />
+          <mesh filename="package://neuronbot2_description/meshes/neuronbot2/top_chassis.dae" />
         </geometry>
       </visual>
@@ -30,5 +30,5 @@
         <visual>
           <geometry>
-            <mesh filename="package://husky_description/meshes/user_rail.dae" />
+            <mesh filename="package://neuronbot2_description/meshes/neuronbot2/user_rail.dae" />
           </geometry>
         </visual>
@@ -45,5 +45,5 @@
       <visual>
         <geometry>
-          <mesh filename="package://husky_description/meshes/bumper.dae" />
+          <mesh filename="package://neuronbot2_description/meshes/neuronbot2/bumper.dae" />
         </geometry>
       </visual>
@@ -59,5 +59,5 @@
           <visual>
               <geometry>
-                  <mesh filename="package://husky_description/meshes/bumper_extension.dae" />
+                  <mesh filename="package://neuronbot2_description/meshes/neuronbot2/bumper_extension.dae" />
               </geometry>
           </visual>
@@ -73,5 +73,5 @@
       <visual>
         <geometry>
-          <mesh filename="package://husky_description/meshes/bumper.dae" />
+          <mesh filename="package://neuronbot2_description/meshes/neuronbot2/bumper.dae" />
         </geometry>
       </visual>
@@ -87,5 +87,5 @@
           <visual>
               <geometry>
-                  <mesh filename="package://husky_description/meshes/bumper_extension.dae" />
+                  <mesh filename="package://neuronbot2_description/meshes/neuronbot2/bumper_extension.dae" />
               </geometry>
           </visual>
@@ -104,5 +104,5 @@
             <origin xyz="0 0 0" rpy="0 0 0" />
             <geometry>
-              <mesh filename="package://husky_description/meshes/large_top_plate.dae" />
+              <mesh filename="package://neuronbot2_description/meshes/neuronbot2/large_top_plate.dae" />
             </geometry>
           </visual>
@@ -110,5 +110,5 @@
             <origin xyz="0 0 0" rpy="0 0 0"/>
             <geometry>
-              <mesh filename="package://husky_description/meshes/large_top_plate_collision.stl" />
+              <mesh filename="package://neuronbot2_description/meshes/neuronbot2/large_top_plate_collision.stl" />
             </geometry>
           </collision>
@@ -138,5 +138,5 @@
             <origin xyz="0 0 0" rpy="0 0 0" />
             <geometry>
-              <mesh filename="package://husky_description/meshes/top_plate.dae" />
+              <mesh filename="package://neuronbot2_description/meshes/neuronbot2/top_plate.dae" />
             </geometry>
           </visual>
@@ -144,5 +144,5 @@
             <origin xyz="0 0 0" rpy="0 0 0"/>
             <geometry>
-              <mesh filename="package://husky_description/meshes/top_plate.stl" />
+              <mesh filename="package://neuronbot2_description/meshes/neuronbot2/top_plate.stl" />
             </geometry>
           </collision>

File: neuronbot2_description/urdf/husky_macro.urdf.xacro (robot description, xacro)
@@ -11,5 +11,5 @@
   <xacro:property name="husky_rear_bumper_extend" value="$(optenv HUSKY_REAR_BUMPER_EXTEND 0)" />
   <xacro:arg name="robot_namespace" default="/" />
-  <xacro:arg name="is_sim" default="false" />
+  <xacro:arg name="is_sim" default="true" />
   <xacro:arg name="urdf_extras" default="$(optenv CPR_URDF_EXTRAS empty.urdf)" />
   <!-- Included URDF/XACRO Files -->

File: neuronbot2_description/urdf/wheel.urdf.xacro (robot description, xacro)
@@ -11,5 +11,5 @@
         <origin xyz="0 0 0" rpy="0 0 0" />
         <geometry>
-          <mesh filename="package://husky_description/meshes/wheel.dae" />
+          <mesh filename="package://neuronbot2_description/meshes/neuronbot2/wheel.dae" />
         </geometry>
       </visual>
