Commit message: added imu plugin

File: neuronbot2_description/urdf/husky_bot.urdf.xacro (robot description, xacro)
@@ -64,11 +64,31 @@
     </joint>
     <!-- IMU Link-->
-    <!-- Can be modified with environment variables in /etc/ros/setup.bash -->
     <link name="imu_link"/>
     <joint name="imu_joint" type="fixed">
-      <origin xyz="$(optenv CPR_IMU_XYZ 0 0 0)" rpy="$(optenv CPR_IMU_RPY 0 0 0)" />
-      <parent link="base_link" />
-      <child link="imu_link" />
+      <parent link="base_link"/>
+      <child link="imu_link"/>
+      <origin xyz="0 0 0" rpy="0 0 0"/>
     </joint>
+    <!-- Gazebo IMU Sensor Plugin -->
+    <gazebo reference="imu_link">
+      <gravity>true</gravity>
+      <sensor name="nb2_imu" type="imu">
+        <always_on>true</always_on>
+        <update_rate>200</update_rate>
+        <visualize>true</visualize>
+        <topic>__default_topic__</topic>
+        <plugin filename="libgazebo_ros_imu_sensor.so" name="neuronbot2_imu">
+          <ros>
+            <remapping>~/out:=imu</remapping>
+          </ros>
+          <gaussianNoise>0.0</gaussianNoise>
+          <xyzOffset>0 0 0</xyzOffset>
+          <rpyOffset>0 0 0</rpyOffset>
+          <!-- <frame_name>imu_link</frame_name> -->
+          <initial_orientation_as_reference>false</initial_orientation_as_reference>
+        </plugin>
+        <pose>0 0 0 0 0 0</pose>
+      </sensor>
+    </gazebo>
     <!-- GPS Link-->
     <!-- Can be modified with environment variables in /etc/ros/setup.bash -->

Commit message: added 2d LiDAR plugin

File: neuronbot2_description/urdf/husky_bot.urdf.xacro (robot description, xacro)
@@ -1,4 +1,7 @@
 <?xml version="1.0"?>
 <robot name="neuronbot2" xmlns:xacro="http://ros.org/wiki/xacro">
+  <material name="Grey">
+    <color rgba="0.5 0.5 0.5 1"/>
+  </material>
   <!-- Included URDF/XACRO Files -->
   <xacro:include filename="$(find neuronbot2_description)/urdf/decorations.urdf.xacro" />
@@ -91,4 +94,66 @@
       </sensor>
     </gazebo>
+    <!-- 2D LiDAR Link -->
+    <link name="laser_frame">
+      <inertial>
+        <mass value="0.125"/>
+        <origin xyz="0 0 0" rpy="0 0 0"/>
+        <inertia ixx="0.001" ixy="0" ixz="0" iyy="0.001" iyz="0" izz="0.001"/>
+      </inertial>
+      <visual>
+        <origin xyz="0 0 0" rpy="0 0 0"/>
+        <geometry>
+          <mesh filename="package://neuronbot2_description/meshes/neuronbot2/laser_link.stl" scale="0.001 0.001 0.001"/>
+        </geometry>
+        <material name="Grey"/>
+      </visual>
+      <collision>
+        <origin xyz="0 0 0" rpy="0 0 0"/>
+        <geometry>
+          <mesh filename="package://neuronbot2_description/meshes/neuronbot2/laser_link.stl" scale="0.001 0.001 0.001"/>
+        </geometry>
+      </collision>
+    </link>
+    <!-- 2D LiDAR Joint (fixed to base_link) -->
+    <joint name="laser_frame_joint" type="fixed">
+      <parent link="base_link"/>
+      <child link="laser_frame"/>
+      <origin xyz="0 0 0.24" rpy="0 0 0"/>
+    </joint>
+    <!-- Gazebo LiDAR Sensor Plugin -->
+    <gazebo reference="laser_frame">
+      <sensor name="rp_lidar_a1" type="ray">
+        <pose>0.0 0 0.02 0 0 0</pose>
+        <update_rate>5.5</update_rate>
+        <visualize>true</visualize>
+        <ray>
+          <scan>
+            <horizontal>
+              <samples>360</samples>
+              <resolution>1.000000</resolution>
+              <min_angle>-3.14</min_angle>
+              <max_angle>3.14</max_angle>
+            </horizontal>
+          </scan>
+          <range>
+            <min>0.2</min>
+            <max>20.0</max>
+            <resolution>0.05</resolution>
+          </range>
+          <noise>
+            <type>gaussian</type>
+            <mean>0.0</mean>
+            <stddev>0.01</stddev>
+          </noise>
+        </ray>
+        <plugin name="neuronbot2_laserscan" filename="libgazebo_ros_ray_sensor.so">
+          <ros>
+            <remapping>~/out:=scan</remapping>
+          </ros>
+          <output_type>sensor_msgs/LaserScan</output_type>
+          <frame_name>laser_frame</frame_name>
+        </plugin>
+      </sensor>
+    </gazebo>
     <!-- GPS Link-->
     <!-- Can be modified with environment variables in /etc/ros/setup.bash -->

Commit message: remove 2d lidar stl

File: neuronbot2_description/urdf/husky_bot.urdf.xacro (robot description, xacro)
@@ -101,5 +101,5 @@
         <inertia ixx="0.001" ixy="0" ixz="0" iyy="0.001" iyz="0" izz="0.001"/>
       </inertial>
-      <visual>
+      <!-- <visual>
         <origin xyz="0 0 0" rpy="0 0 0"/>
         <geometry>
@@ -107,11 +107,11 @@
         </geometry>
         <material name="Grey"/>
-      </visual>
-      <collision>
+      </visual> -->
+      <!-- <collision>
         <origin xyz="0 0 0" rpy="0 0 0"/>
         <geometry>
           <mesh filename="package://neuronbot2_description/meshes/neuronbot2/laser_link.stl" scale="0.001 0.001 0.001"/>
         </geometry>
-      </collision>
+      </collision> -->
     </link>
     <!-- 2D LiDAR Joint (fixed to base_link) -->
@@ -138,5 +138,5 @@
           <range>
             <min>0.2</min>
-            <max>20.0</max>
+            <max>10.0</max>
             <resolution>0.05</resolution>
           </range>

Commit message: added livox sense and cleaned rviz2

File: neuronbot2_description/urdf/husky_bot.urdf.xacro (robot description, xacro)
@@ -10,4 +10,5 @@
   <!-- <xacro:include filename="$(find neuronbot2_description)/urdf/accessories/sick_lms1xx_mount.urdf.xacro"/> -->
   <xacro:include filename="$(find neuronbot2_description)/urdf/accessories/sensor_arch.urdf.xacro"/>
+  <xacro:include filename="$(find ros2_livox_simulation)/urdf/mid360.xacro" /> <!-- 여기에 추가 -->
   <xacro:property name="M_PI" value="3.14159"/>
   <xacro:property name="husky_front_bumper_extend" value="$(optenv HUSKY_FRONT_BUMPER_EXTEND 0)" />
@@ -191,4 +192,8 @@
       <origin xyz="${-wheelbase/2} ${-track/2} ${wheel_vertical_offset}" rpy="0 0 0" />
     </xacro:husky_wheel>
+    <!-- Livox MID-360 센서 추가 (로봇 중심 위 z=0.3m에 장착) -->
+    <xacro:mid360 name="livox" parent="base_link" topic="mid360">
+      <origin xyz="0 0 0.3" rpy="0 0 0"/>
+    </xacro:mid360>
     <xacro:husky_decorate />
   </xacro:macro>
